Commit message: package working on gazebo

File: iiwa_description/urdf/kuka14.urdf (robot description, URDF)
Before this commit: robot iiwa14, 10 links, 9 joints
Links:
- link iiwa_link_0: geometry collision mesh filename=package://iit-iiwa-ros-pkg/iiwa_description/meshes/iiwa14/c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; visual mesh filename=package://iit-iiwa-ros-pkg/iiwa_description/meshes/iiwa14/v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
- link iiwa_link_1: geometry collision mesh filename=package://iit-iiwa-ros-pkg/iiwa_description/meshes/iiwa14/c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; visual mesh filename=package://iit-iiwa-ros-pkg/iiwa_description/meshes/iiwa14/v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
- link iiwa_link_2: geometry collision mesh filename=package://iit-iiwa-ros-pkg/iiwa_description/meshes/iiwa14/c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; visual mesh filename=package://iit-iiwa-ros-pkg/iiwa_description/meshes/iiwa14/v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
- link iiwa_link_3: geometry collision mesh filename=package://iit-iiwa-ros-pkg/iiwa_description/meshes/iiwa14/c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; visual mesh filename=package://iit-iiwa-ros-pkg/iiwa_description/meshes/iiwa14/v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
- link iiwa_link_4: geometry collision mesh filename=package://iit-iiwa-ros-pkg/iiwa_description/meshes/iiwa14/c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; visual mesh filename=package://iit-iiwa-ros-pkg/iiwa_description/meshes/iiwa14/v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
- link iiwa_link_5: geometry collision mesh filename=package://iit-iiwa-ros-pkg/iiwa_description/meshes/iiwa14/c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; visual mesh filename=package://iit-iiwa-ros-pkg/iiwa_description/meshes/iiwa14/v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
- link iiwa_link_6: geometry collision mesh filename=package://iit-iiwa-ros-pkg/iiwa_description/meshes/iiwa14/c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; visual mesh filename=package://iit-iiwa-ros-pkg/iiwa_description/meshes/iiwa14/v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
- link iiwa_link_7: geometry collision mesh filename=package://iit-iiwa-ros-pkg/iiwa_description/meshes/iiwa14/c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; visual mesh filename=package://iit-iiwa-ros-pkg/iiwa_description/meshes/iiwa14/v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

File: iiwa_description/urdf/kuka7.urdf (robot description, URDF)
Before this commit: robot iiwa7, 10 links, 9 joints
Links:
- link iiwa_link_0: geometry collision mesh filename=package://iit-iiwa-ros-pkg/iiwa_description/meshes/iiwa7/co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; visual mesh filename=package://iit-iiwa-ros-pkg/iiwa_description/meshes/iiwa7/vi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
- link iiwa_link_1: geometry collision mesh filename=package://iit-iiwa-ros-pkg/iiwa_description/meshes/iiwa7/co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; visual mesh filename=package://iit-iiwa-ros-pkg/iiwa_description/meshes/iiwa7/vi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
- link iiwa_link_2: geometry collision mesh filename=package://iit-iiwa-ros-pkg/iiwa_description/meshes/iiwa7/co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; visual mesh filename=package://iit-iiwa-ros-pkg/iiwa_description/meshes/iiwa7/vi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
- link iiwa_link_3: geometry collision mesh filename=package://iit-iiwa-ros-pkg/iiwa_description/meshes/iiwa7/co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; visual mesh filename=package://iit-iiwa-ros-pkg/iiwa_description/meshes/iiwa7/vi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
- link iiwa_link_4: geometry collision mesh filename=package://iit-iiwa-ros-pkg/iiwa_description/meshes/iiwa7/co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; visual mesh filename=package://iit-iiwa-ros-pkg/iiwa_description/meshes/iiwa7/vi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
- link iiwa_link_5: geometry collision mesh filename=package://iit-iiwa-ros-pkg/iiwa_description/meshes/iiwa7/co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; visual mesh filename=package://iit-iiwa-ros-pkg/iiwa_description/meshes/iiwa7/vi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
- link iiwa_link_6: geometry collision mesh filename=package://iit-iiwa-ros-pkg/iiwa_description/meshes/iiwa7/co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; visual mesh filename=package://iit-iiwa-ros-pkg/iiwa_description/meshes/iiwa7/vi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
- link iiwa_link_7: geometry collision mesh filename=package://iit-iiwa-ros-pkg/iiwa_description/meshes/iiwa7/co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; visual mesh filename=package://iit-iiwa-ros-pkg/iiwa_description/meshes/iiwa7/vi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
